File: Beacon Detector/IR_BEACON.sch (EAGLE design)
At the start: 38 parts, among them U1 LP2950-3.0ACZ

Commit message: Added more to the beacon detector and finished the ring gears.
Connections:
- removed net V_OUT: J2.1, R25.2, R28.1, R6.2
- net N$1: now also D3.A, R1.2, R3.2, U$1.VIND-; no longer R1.1
- net VOUTC: now also J2.1, R25.2, R28.1, R6.2
- net V_BIAS: now also U$1.VIND+
- net V_FILT: now also R1.1; no longer D3.A, R1.2, R3.2
Changed lines of the file:
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@@
 <pinref part="U$1" gate="A" pin="VDD"/>
 <pinref part="P+2" gate="1" pin="VCC"/>
+<junction x="264.16" y="111.76"/>
 </segment>
 <segment>
@@
 <pinref part="U$1" gate="A" pin="VSS"/>
 <pinref part="GND4" gate="1" pin="GND"/>
+<junction x="312.42" y="111.76"/>
 </segment>
 <segment>
@@
 <wire x1="254" y1="144.78" x2="254" y2="119.38" width="0.1524" layer="91"/>
 <pinref part="1K" gate="G$1" pin="S"/>
+<junction x="264.16" y="119.38"/>
+<junction x="264.16" y="116.84"/>
 </segment>
 <segment>
@@
 <wire x1="325.12" y1="114.3" x2="312.42" y2="114.3" width="0.1524" layer="91"/>
 <label x="337.82" y="114.3" size="1.778" layer="95"/>
+<pinref part="U$1" gate="A" pin="VIND+"/>
+<junction x="312.42" y="114.3"/>
 </segment>
 </net>
@@
 <wire x1="259.08" y1="73.66" x2="256.54" y2="73.66" width="0.1524" layer="91"/>
 <wire x1="203.2" y1="91.44" x2="259.08" y2="91.44" width="0.1524" layer="91"/>
+<junction x="264.16" y="106.68"/>
 </segment>
 </net>
@@
 <junction x="170.18" y="101.6"/>
 <pinref part="10K" gate="G$1" pin="S"/>
-</segment>
-<segment>
-<pinref part="R1" gate="G$1" pin="2"/>
-<wire x1="325.12" y1="116.84" x2="322.58" y2="116.84" width="0.1524" layer="91"/>
-<label x="337.82" y="116.84" size="1.778" layer="95"/>
-<pinref part="D3" gate="G$1" pin="A"/>
-<wire x1="322.58" y1="116.84" x2="317.5" y2="116.84" width="0.1524" layer="91"/>
-<wire x1="317.5" y1="116.84" x2="312.42" y2="116.84" width="0.1524" layer="91"/>
-<junction x="317.5" y="116.84"/>
-<pinref part="R3" gate="G$1" pin="2"/>
-<junction x="322.58" y="116.84"/>
+<junction x="264.16" y="104.14"/>
+</segment>
+<segment>
+<pinref part="R1" gate="G$1" pin="1"/>
+<wire x1="335.28" y1="116.84" x2="345.44" y2="116.84" width="0.2032" layer="91"/>
 </segment>
 </net>
@@
 </segment>
 </net>
-<net name="V_OUT" class="0">
-<segment>
-<pinref part="J2" gate="G$1" pin="1"/>
-<wire x1="38.1" y1="154.94" x2="38.1" y2="152.4" width="0.1524" layer="91"/>
-<label x="38.1" y="147.32" size="1.778" layer="95" rot="R90"/>
-</segment>
-<segment>
-<label x="307.34" y="68.58" size="1.778" layer="95" rot="R180"/>
-<pinref part="R25" gate="G$1" pin="2"/>
-<pinref part="R6" gate="G$1" pin="2"/>
-<wire x1="314.96" y1="68.58" x2="309.88" y2="68.58" width="0.1524" layer="91"/>
-<wire x1="309.88" y1="68.58" x2="307.34" y2="68.58" width="0.1524" layer="91"/>
-<wire x1="314.96" y1="48.26" x2="314.96" y2="68.58" width="0.1524" layer="91"/>
-<pinref part="R28" gate="G$1" pin="1"/>
-<junction x="309.88" y="68.58"/>
-</segment>
-</net>
 <net name="V_IN" class="0">
 <segment>
@@
 <wire x1="264.16" y1="114.3" x2="215.9" y2="114.3" width="0.1524" layer="91"/>
 <pinref part="C2" gate="G$1" pin="+"/>
+<junction x="264.16" y="114.3"/>
 </segment>
 </net>
@@
 <pinref part="U$1" gate="A" pin="VINB+"/>
 <wire x1="254" y1="109.22" x2="264.16" y2="109.22" width="0.1524" layer="91"/>
+<junction x="264.16" y="109.22"/>
 </segment>
 </net>
@@
 </segment>
 </net>
-<net name="N$1" class="0">
-<segment>
-<pinref part="R1" gate="G$1" pin="1"/>
-<wire x1="345.44" y1="116.84" x2="335.28" y2="116.84" width="0.2032" layer="91"/>
-</segment>
-</net>
 <net name="N$2" class="0">
 <segment>
 <pinref part="R2" gate="G$1" pin="1"/>
 <wire x1="335.28" y1="114.3" x2="345.44" y2="114.3" width="0.2032" layer="91"/>
+<junction x="335.28" y="114.3"/>
 </segment>
 </net>
@@
 <pinref part="D4" gate="G$1" pin="A"/>
 <junction x="312.42" y="121.92"/>
+<junction x="312.42" y="119.38"/>
 </segment>
 </net>
@@
 <pinref part="C1" gate="G$1" pin="+"/>
 <junction x="312.42" y="149.86"/>
+<junction x="312.42" y="106.68"/>
 </segment>
 </net>
@@
 <wire x1="327.66" y1="109.22" x2="312.42" y2="109.22" width="0.1524" layer="91"/>
 <label x="327.66" y="109.22" size="1.778" layer="95"/>
+<junction x="312.42" y="109.22"/>
 </segment>
 </net>
@@
 <wire x1="312.42" y1="104.14" x2="327.66" y2="104.14" width="0.1524" layer="91"/>
 <label x="327.66" y="104.14" size="1.778" layer="95"/>
+<junction x="312.42" y="104.14"/>
+</segment>
+<segment>
+<pinref part="J2" gate="G$1" pin="1"/>
+<wire x1="38.1" y1="154.94" x2="38.1" y2="152.4" width="0.1524" layer="91"/>
+<label x="38.1" y="147.32" size="1.778" layer="95" rot="R90"/>
+</segment>
+<segment>
+<label x="307.34" y="68.58" size="1.778" layer="95" rot="R180"/>
+<pinref part="R25" gate="G$1" pin="2"/>
+<pinref part="R6" gate="G$1" pin="2"/>
+<wire x1="314.96" y1="68.58" x2="309.88" y2="68.58" width="0.1524" layer="91"/>
+<wire x1="309.88" y1="68.58" x2="307.34" y2="68.58" width="0.1524" layer="91"/>
+<wire x1="314.96" y1="48.26" x2="314.96" y2="68.58" width="0.1524" layer="91"/>
+<pinref part="R28" gate="G$1" pin="1"/>
+<junction x="309.88" y="68.58"/>
 </segment>
 </net>
@@
 </segment>
 </net>
+<net name="N$1" class="0">
+<segment>
+<pinref part="U$1" gate="A" pin="VIND-"/>
+<pinref part="D3" gate="G$1" pin="A"/>
+<wire x1="312.42" y1="116.84" x2="317.5" y2="116.84" width="0.2032" layer="91"/>
+<pinref part="R3" gate="G$1" pin="2"/>
+<wire x1="317.5" y1="116.84" x2="322.58" y2="116.84" width="0.2032" layer="91"/>
+<pinref part="R1" gate="G$1" pin="2"/>
+<wire x1="322.58" y1="116.84" x2="325.12" y2="116.84" width="0.2032" layer="91"/>
+<junction x="312.42" y="116.84"/>
+</segment>
+</net>

Commit message: Finished Beacon Detector.
Parts:
- removed JP4: STAND-OFFTIGHT, ASL:STAND-OFFTIGHT
Connections:
- removed net N$17: D4.C, R3.1
- net V_ENV1: now also D4.C, R3.1
Changed lines of the file:
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@@
 <part name="JP5" library="ASL" deviceset="STAND-OFF" device="TIGHT"/>
 <part name="JP3" library="ASL" deviceset="STAND-OFF" device="TIGHT"/>
-<part name="JP4" library="ASL" deviceset="STAND-OFF" device="TIGHT"/>
 <part name="C7" library="ASL" deviceset="CAP" device="0805" value=".1uF"/>
 <part name="U1" library="ASL" deviceset="LP2950" device="ACZ" technology="-3.0"/>
@@
 <instance part="JP5" gate="G$1" x="20.32" y="162.56"/>
 <instance part="JP3" gate="G$1" x="27.94" y="162.56"/>
-<instance part="JP4" gate="G$1" x="30.48" y="162.56"/>
 <instance part="C7" gate="G$1" x="55.88" y="154.94"/>
 <instance part="U1" gate="G$1" x="63.5" y="134.62"/>
@@
 <wire x1="337.82" y1="35.56" x2="314.96" y2="35.56" width="0.1524" layer="91"/>
 <wire x1="337.82" y1="35.56" x2="337.82" y2="33.02" width="0.1524" layer="91"/>
+<junction x="337.82" y="35.56"/>
 </segment>
 </net>
@@
 <pinref part="C8" gate="G$1" pin="2"/>
 <wire x1="63.5" y1="127" x2="71.12" y2="127" width="0.1524" layer="91"/>
+<junction x="63.5" y="127"/>
 </segment>
 <segment>
@@
 <junction x="264.16" y="119.38"/>
 <junction x="264.16" y="116.84"/>
+<junction x="254" y="119.38"/>
+<junction x="157.48" y="139.7"/>
 </segment>
 <segment>
@@
 <pinref part="U$1" gate="A" pin="VIND+"/>
 <junction x="312.42" y="114.3"/>
+<junction x="325.12" y="114.3"/>
 </segment>
 </net>
@@
 <wire x1="223.52" y1="73.66" x2="213.36" y2="73.66" width="0" layer="91"/>
 <pinref part="R24" gate="G$1" pin="1"/>
+<junction x="213.36" y="73.66"/>
 </segment>
 </net>
@@
 <wire x1="203.2" y1="91.44" x2="259.08" y2="91.44" width="0.1524" layer="91"/>
 <junction x="264.16" y="106.68"/>
+<junction x="259.08" y="91.44"/>
 </segment>
 </net>
@@
 <pinref part="R1" gate="G$1" pin="1"/>
 <wire x1="335.28" y1="116.84" x2="345.44" y2="116.84" width="0.2032" layer="91"/>
+<junction x="335.28" y="116.84"/>
+<label x="337.82" y="116.84" size="1.778" layer="95"/>
 </segment>
 </net>
@@
 <pinref part="C2" gate="G$1" pin="+"/>
 <junction x="264.16" y="114.3"/>
+<junction x="215.9" y="114.3"/>
 </segment>
 </net>
@@
 </segment>
 </net>
-<net name="N$17" class="0">
-<segment>
-<pinref part="R3" gate="G$1" pin="1"/>
-<pinref part="D4" gate="G$1" pin="C"/>
-<wire x1="322.58" y1="127" x2="312.42" y2="127" width="0.1524" layer="91"/>
-<wire x1="312.42" y1="127" x2="312.42" y2="132.08" width="0.1524" layer="91"/>
-</segment>
-</net>
 <net name="V_ENV1" class="0">
 <segment>
-<wire x1="312.42" y1="132.08" x2="312.42" y2="149.86" width="0.1524" layer="91"/>
 <pinref part="R5" gate="G$1" pin="1"/>
 <wire x1="312.42" y1="149.86" x2="312.42" y2="157.48" width="0.1524" layer="91"/>
@@
 <wire x1="353.06" y1="106.68" x2="312.42" y2="106.68" width="0.1524" layer="91"/>
 <pinref part="C1" gate="G$1" pin="+"/>
+<junction x="312.42" y="106.68"/>
+<pinref part="R3" gate="G$1" pin="1"/>
+<pinref part="D4" gate="G$1" pin="C"/>
+<wire x1="322.58" y1="127" x2="312.42" y2="127" width="0.1524" layer="91"/>
+<wire x1="312.42" y1="127" x2="312.42" y2="149.86" width="0.2032" layer="91"/>
+<junction x="312.42" y="127"/>
 <junction x="312.42" y="149.86"/>
-<junction x="312.42" y="106.68"/>
+<junction x="312.42" y="157.48"/>
 </segment>
 </net>
@@
 <wire x1="353.06" y1="48.26" x2="353.06" y2="66.04" width="0.1524" layer="91"/>
 <label x="350.52" y="66.04" size="1.778" layer="95"/>
+<junction x="353.06" y="48.26"/>
 </segment>
 <segment>
@@
 <pinref part="R28" gate="G$1" pin="1"/>
 <junction x="309.88" y="68.58"/>
+<junction x="314.96" y="48.26"/>
 </segment>
 </net>
@@
 <wire x1="322.58" y1="116.84" x2="325.12" y2="116.84" width="0.2032" layer="91"/>
 <junction x="312.42" y="116.84"/>
-</segment>
-</net>
+<junction x="322.58" y="116.84"/>
+<junction x="317.5" y="116.84"/>
+</segment>
+</net>
